File: Quest_EMG/_autosave-untitled.kicad_sch (KiCad schematic)
At the start: 42 parts, among them IC1 OPA2890IDGST, U1 AD8620, U2 INA121UAE4

Commit message: feature amplification
Connections:
- net 33: now also IC1.7 (OUT_B); no longer IC1.6 (-IN_B), R8.1
- net at R8.2: now also IC1.6 (-IN_B), R8.1; no longer IC1.7 (OUT_B)
Other:
- moved on the sheet: R8
Changed lines of the file:
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@@
   (junction (at 210.82 113.03) (diameter 0) (color 0 0 0 0)
   )
-  (junction (at 214.63 120.65) (diameter 0) (color 0 0 0 0)
-  )
-  (junction (at 214.63 118.11) (diameter 0) (color 0 0 0 0)
-  )
   (junction (at 46.99 54.61) (diameter 0) (color 0 0 0 0)
   )
@@
   (junction (at 78.74 68.58) (diameter 0) (color 0 0 0 0)
   )
+  (junction (at 210.82 120.65) (diameter 0) (color 0 0 0 0)
+  )
+  (junction (at 220.98 118.11) (diameter 0) (color 0 0 0 0)
+  )
   (junction (at 157.48 163.83) (diameter 0) (color 0 0 0 0)
   )
@@
     (stroke (width 0) (type default))
   )
-  (wire (pts (xy 214.63 118.11) (xy 214.63 120.65))
+  (wire (pts (xy 220.98 125.73) (xy 210.82 125.73))
     (stroke (width 0) (type default))
   )
@@
     (stroke (width 0) (type default))
   )
-  (wire (pts (xy 214.63 118.11) (xy 234.95 118.11))
+  (wire (pts (xy 201.93 118.11) (xy 220.98 118.11))
     (stroke (width 0) (type default))
   )
@@
     (stroke (width 0) (type default))
   )
-  (wire (pts (xy 209.55 118.11) (xy 214.63 118.11))
-    (stroke (width 0) (type default))
-  )
   (wire (pts (xy 201.93 110.49) (xy 203.2 110.49))
     (stroke (width 0) (type default))
@@
     (stroke (width 0) (type default))
   )
-  (wire (pts (xy 201.93 120.65) (xy 214.63 120.65))
+  (wire (pts (xy 201.93 120.65) (xy 210.82 120.65))
     (stroke (width 0) (type default))
   )
@@
     (stroke (width 0) (type default))
   )
+  (wire (pts (xy 210.82 120.65) (xy 210.82 125.73))
+    (stroke (width 0) (type default))
+  )
   (wire (pts (xy 214.63 53.34) (xy 218.44 53.34))
     (stroke (width 0) (type default))
@@
     (stroke (width 0) (type default))
   )
+  (wire (pts (xy 220.98 118.11) (xy 234.95 118.11))
+    (stroke (width 0) (type default))
+  )
   (wire (pts (xy 168.91 53.34) (xy 168.91 60.96))
     (stroke (width 0) (type default))
@@
     (stroke (width 0) (type default))
   )
+  (wire (pts (xy 210.82 120.65) (xy 218.44 120.65))
+    (stroke (width 0) (type default))
+  )
   (wire (pts (xy 156.21 119.38) (xy 154.94 119.38))
     (stroke (width 0) (type default))
@@
   )
   (wire (pts (xy 99.06 120.65) (xy 107.95 120.65))
-    (stroke (width 0) (type default))
-  )
-  (wire (pts (xy 214.63 120.65) (xy 218.44 120.65))
     (stroke (width 0) (type default))
   )
@@
     )
   )
-  (symbol (lib_id "Device:R") (at 205.74 118.11 270) (unit 1)
-    (in_bom yes) (on_board yes) (dnp no)
-    (property "Reference" "R8" (at 203.2 120.65 90)
-      (effects (font (size 1.27 1.27)) (justify left))
-    )
-    (property "Value" "15K" (at 207.01 120.65 90)
-      (effects (font (size 1.27 1.27)) (justify left))
-    )
-    (property "Footprint" "Resistor_SMD:R_0402_1005Metric" (at 205.74 116.332 90)
-      (effects (font (size 1.27 1.27)) hide)
-    )
-    (property "Datasheet" "~" (at 205.74 118.11 0)
-      (effects (font (size 1.27 1.27)) hide)
-    )
+  (symbol (lib_id "Device:R") (at 220.98 121.92 0) (unit 1)
+    (in_bom yes) (on_board yes) (dnp no)
+    (property "Reference" "R8" (at 223.52 123.19 0)
+      (effects (font (size 1.27 1.27)) (justify left))
+    )
+    (property "Value" "15K" (at 223.52 120.65 0)
+      (effects (font (size 1.27 1.27)) (justify left))
+    )
+    (property "Footprint" "Resistor_SMD:R_0402_1005Metric" (at 219.202 121.92 90)
+      (effects (font (size 1.27 1.27)) hide)
+    )
+    (property "Datasheet" "~" (at 220.98 121.92 0)
+      (effects (font (size 1.27 1.27)) hide)
+    )
