File: Quest_EMG/Quest_EMG.kicad_sch (KiCad schematic)
At the start: 3 parts

Commit message: forgot something
Changed lines of the file:
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@@
     (fill (type none))
   )
-  (text_box "TO DO:\n*amplify signal to 1,65V from 45uV\n*offset signal bij 1,65V\n*Add charging capabilities\n*add screwholes"
+  (text_box "TO DO:\n*add filters\n*add charging capabilities\n*add screwholes"
     (at 228.6 63.5 0) (size 46.99 76.2)
     (stroke (width 0) (type default))
